File: PCB/Tao Te Ching.kicad_pcb (KiCad board)
At the start: 2 copper layers, 278.3 x 93.1 mm, 101 parts, among them SW1 SW_Push_45deg, SW10 SW_Push_45deg, SW11 SW_Push_45deg, SW12 SW_Push_45deg, SW13 SW_Push_45deg, SW14 SW_Push_45deg, SW15 SW_Push_45deg, SW16 SW_Push_45deg, SW17 SW_Push_45deg, SW18 SW_Push_45deg, SW19 SW_Push_45deg, SW2 SW_Push_45deg, SW20 SW_Push_45deg, SW21 SW_Push_45deg, SW22 SW_Push_45deg, SW23 SW_Push_45deg, SW24 SW_Push_45deg, SW25 SW_Push_45deg, SW26 SW_Push_45deg, SW27 SW_Push_45deg, SW28 SW_Push_45deg, SW29 SW_Push_45deg, SW3 SW_Push_45deg, SW30 SW_Push_45deg, SW31 SW_Push_45deg, SW32 SW_Push_45deg, SW33 SW_Push_45deg, SW34 SW_Push_45deg, SW35 SW_Push_45deg, SW36 SW_Push_45deg, SW37 SW_Push_45deg, SW38 SW_Push_45deg, SW39 SW_Push_45deg, SW4 SW_Push_45deg, SW40 SW_Push_45deg, SW41 SW_Push_45deg, SW42 SW_Push_45deg, SW43 SW_Push_45deg, SW44 SW_Push_45deg, SW45 SW_Push_45deg, SW46 SW_Push_45deg, SW47 SW_Push_45deg, SW48 SW_Push_45deg, SW5 SW_Push_45deg, SW6 SW_Push_45deg, SW7 SW_Push_45deg, SW8 SW_Push_45deg, SW9 SW_Push_45deg, U1 XIAO-nRF52840-DIP, U2 XIAO-nRF52840-DIP

Commit message: Updated PCB and Added /Images
Routing:
- net Col0: track 0.00 -> 196.7 mm
- net Col11: track 0.00 -> 184.4 mm, vias 0 -> 2
- net Col1: track 0.00 -> 169.1 mm
- net Row0: track 0.00 -> 168.8 mm
- net Row4: track 0.00 -> 167.7 mm, vias 0 -> 1
- net Col10: track 0.00 -> 160.3 mm, vias 0 -> 1
- net Row5: track 0.00 -> 150.7 mm
- net Row1: track 0.00 -> 150.2 mm
- net Col2: track 0.00 -> 148.8 mm
- net Col9: track 0.00 -> 148.3 mm, vias 0 -> 1
- net Col8: track 0.00 -> 148.2 mm, vias 0 -> 3
- net Row7: track 0.00 -> 144.9 mm, vias 0 -> 1
- net Col3: track 0.00 -> 144.4 mm, vias 0 -> 1
- net Row6: track 0.00 -> 134.6 mm, vias 0 -> 1
- net Row2: track 0.00 -> 130.0 mm
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
Commit message: Reworked Case and images
Parts:
- moved U1 0.19 mm to (276.5, 123.2)
- moved SW18 0.11 mm to (258.7, 99.6)
- moved SW24 0.11 mm to (258.7, 118.6)
- moved SW6 0.11 mm to (258.7, 61.5)
- moved SW12 0.11 mm to (258.7, 80.5)
- moved D10 0.11 mm to (210.2, 76.1)
- moved D16 0.11 mm to (210.2, 95.2)
- moved D19 0.11 mm to (152.7, 124.6)
- moved D2 0.11 mm to (172.1, 64.2)
- moved D20 0.11 mm to (172.1, 121.3)
- moved D8 0.11 mm to (172.1, 83.2)
- moved SW11 0.11 mm to (239.7, 75.8)
- moved SW20 0.11 mm to (182.5, 115.5)
- moved SW23 0.11 mm to (239.7, 113.9)
- moved D4 0.11 mm to (210.2, 57.1)
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Routing:
- net Row0: track 168.8 -> 187.0 mm
- net Col4: track 120.3 -> 133.7 mm, vias 1 -> 0
- net Col0: track 196.7 -> 185.7 mm, vias 0 -> 1
- net Col5: track 96.7 -> 107.5 mm, vias 1 -> 0
- net Row1: track 150.2 -> 142.9 mm
- net Col2: track 148.8 -> 155.7 mm, vias 0 -> 1
- net Col3: track 144.4 -> 147.7 mm
- net Row5: track 150.7 -> 152.8 mm
- net Col1: track 169.1 -> 170.5 mm, vias 0 -> 1
- net Row3: track 125.0 -> 126.0 mm
- net Row2: track 130.0 -> 130.9 mm
- net Col11: track 184.4 -> 185.1 mm
- net Row6: track 134.6 -> 135.1 mm
Other:
- board size 278.3 x 93.1 mm -> 278.2 x 89.7 mm

Commit message: Added silkscreen art
Parts:
- added G***: LOGO, LOGO, F.Cu at (21.8, 123.0)
- added G***: LOGO, LOGO, B.Cu at (161.0, 73.5)
- added G***: LOGO, LOGO, B.Cu at (217.9, 62.0)
- added G***: LOGO, LOGO, B.Cu at (199.6, 84.1)
- added G***: LOGO, LOGO, F.Cu at (276.9, 123.1)
- added G***: LOGO, LOGO, B.Cu at (97.2, 85.9)
- added G***: LOGO, LOGO, B.Cu at (164.1, 113.8)
- added G***: LOGO, LOGO, B.Cu at (136.9, 73.4)
- added G***: LOGO, LOGO, B.Cu at (51.5, 87.3)
- added G***: LOGO, LOGO, B.Cu at (133.9, 113.4)
- added G***: LOGO, LOGO, B.Cu at (80.3, 60.5)
- added G***: LOGO, LOGO, B.Cu at (243.1, 87.8)
Other:
- board text added: "TAO TE CHING"
- board text added: "sudo-apt-install-tap"
