File: PCB/Tao Te Ching.kicad_pcb (KiCad board)
At the start: 2 copper layers, 278.2 x 89.7 mm, 113 parts, among them SW1 SW_Push_45deg, SW10 SW_Push_45deg, SW11 SW_Push_45deg, SW12 SW_Push_45deg, SW13 SW_Push_45deg, SW14 SW_Push_45deg, SW15 SW_Push_45deg, SW16 SW_Push_45deg, SW17 SW_Push_45deg, SW18 SW_Push_45deg, SW19 SW_Push_45deg, SW2 SW_Push_45deg, SW20 SW_Push_45deg, SW21 SW_Push_45deg, SW22 SW_Push_45deg, SW23 SW_Push_45deg, SW24 SW_Push_45deg, SW25 SW_Push_45deg, SW26 SW_Push_45deg, SW27 SW_Push_45deg, SW28 SW_Push_45deg, SW29 SW_Push_45deg, SW3 SW_Push_45deg, SW30 SW_Push_45deg, SW31 SW_Push_45deg, SW32 SW_Push_45deg, SW33 SW_Push_45deg, SW34 SW_Push_45deg, SW35 SW_Push_45deg, SW36 SW_Push_45deg, SW37 SW_Push_45deg, SW38 SW_Push_45deg, SW39 SW_Push_45deg, SW4 SW_Push_45deg, SW40 SW_Push_45deg, SW41 SW_Push_45deg, SW42 SW_Push_45deg, SW43 SW_Push_45deg, SW44 SW_Push_45deg, SW45 SW_Push_45deg, SW46 SW_Push_45deg, SW47 SW_Push_45deg, SW48 SW_Push_45deg, SW5 SW_Push_45deg, SW6 SW_Push_45deg, SW7 SW_Push_45deg, SW8 SW_Push_45deg, SW9 SW_Push_45deg, U1 XIAO-nRF52840-DIP, U2 XIAO-nRF52840-DIP

Commit message: Added hotswap sockets
Parts:
- D1, D10, D11, D12, D13, D14, D15, D16, D17, D18, D19, D2, D20, D21, D22, D23, D24, D25, D26, D27, D28, D29, D3, D30, D31, D32, D33, D34, D35, D36, D37, D38, D39, D4, D40, D41, D42, D43, D44, D45, D46, D47, D48, D5, D6, D7, D8, D9: moved to B.Cu
- SW1, SW10, SW11, SW12, SW13, SW14, SW15, SW16, SW17, SW18, SW19, SW2, SW20, SW21, SW22, SW23, SW24, SW25, SW26, SW27, SW28, SW29, SW3, SW30, SW31, SW32, SW33, SW34, SW35, SW36, SW37, SW38, SW39, SW4, SW40, SW41, SW42, SW43, SW44, SW45, SW46, SW47, SW48, SW5, SW6, SW7, SW8, SW9: footprint Taps Keyboard shit:SW_Cherry_MX_1.00u_PCB -> KEYS:SW_Hotswap_Kailh_MX
- moved D29 17.4 mm to (69.8, 61.9)
- moved D45 17.4 mm to (145.9, 66.6)
- moved D13 17.2 mm to (169.6, 104.3)
- moved D27 17.2 mm to (50.5, 104.3)
- moved D39 17.2 mm to (107.4, 96.6)
- moved D46 17.1 mm to (145.7, 85.7)
- moved D1 17.1 mm to (169.9, 66.4)
- moved D44 17.1 mm to (126.5, 120.3)
- moved D37 17.1 mm to (107.5, 58.6)
- moved D33 17.0 mm to (88.4, 56.0)
- moved D47 17.0 mm to (145.6, 104.7)
- moved D34 17.0 mm to (88.4, 75.3)
- moved D41 17.0 mm to (126.5, 63.4)
- moved D38 17.0 mm to (107.5, 77.5)
- moved D35 17.0 mm to (88.4, 94.3)
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Routing:
- net Col11: track 185.1 -> 246.4 mm, vias 2 -> 7
- net Row0: track 187.0 -> 157.5 mm
- net Col2: track 155.7 -> 183.3 mm, vias 1 -> 7
- net Col8: track 148.5 -> 125.2 mm, vias 3 -> 8
- net Col0: track 185.7 -> 202.8 mm
- net Row6: track 135.1 -> 150.9 mm, vias 1 -> 2
- net Row3: track 126.0 -> 110.4 mm
- net Col1: track 170.5 -> 186.0 mm, vias 1 -> 0
- net Col6: track 99.3 -> 84.4 mm, vias 1 -> 2
- net Col9: track 148.3 -> 133.9 mm, vias 1 -> 9
- net Row4: track 167.7 -> 181.8 mm, vias 1 -> 2
- net Col10: track 160.3 -> 147.7 mm, vias 1 -> 5
- net Col7: track 120.7 -> 109.6 mm, vias 0 -> 4
- net Row5: track 152.8 -> 163.5 mm
- net Col5: track 107.5 -> 97.6 mm, vias 0 -> 6
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