File: PCB/Right Sheet.kicad_sch (KiCad schematic)
At the start: 49 parts, among them SW25 SW_Push_45deg, SW26 SW_Push_45deg, SW27 SW_Push_45deg, SW28 SW_Push_45deg, SW29 SW_Push_45deg, SW30 SW_Push_45deg, SW31 SW_Push_45deg, SW32 SW_Push_45deg, SW33 SW_Push_45deg, SW34 SW_Push_45deg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

Commit message: Added hotswap sockets
Parts:
- SW25, SW26, SW27, SW28, SW29, SW30, SW31, SW32, SW33, SW34, SW35, SW36, SW37, SW38, SW39, SW40, SW41, SW42, SW43, SW44, SW45, SW46, SW47, SW48: footprint Taps Keyboard shit:SW_Cherry_MX_1.00u_PCB -> KEYS:SW_Hotswap_Kailh_MX
Changed lines of the file:
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@@
 			)
 		)
-		(property "Footprint" "Taps Keyboard shit:SW_Cherry_MX_1.00u_PCB"
+		(property "Footprint" "KEYS:SW_Hotswap_Kailh_MX"
 			(at 39.37 39.37 0)
 			(effects
@@
 			)
 		)
-		(property "Footprint" "Taps Keyboard shit:SW_Cherry_MX_1.00u_PCB"
+		(property "Footprint" "KEYS:SW_Hotswap_Kailh_MX"
 			(at 100.33 59.69 0)
 			(effects
@@
 			)
 		)
-		(property "Footprint" "Taps Keyboard shit:SW_Cherry_MX_1.00u_PCB"
+		(property "Footprint" "KEYS:SW_Hotswap_Kailh_MX"
 			(at 115.57 39.37 0)
 			(effects
@@
 			)
 		)
-		(property "Footprint" "Taps Keyboard shit:SW_Cherry_MX_1.00u_PCB"
+		(property "Footprint" "KEYS:SW_Hotswap_Kailh_MX"
 			(at 100.33 80.01 0)
 			(effects
@@
 			)
 		)
-		(property "Footprint" "Taps Keyboard shit:SW_Cherry_MX_1.00u_PCB"
+		(property "Footprint" "KEYS:SW_Hotswap_Kailh_MX"
 			(at 69.85 59.69 0)
 			(effects
@@
 			)
 		)
-		(property "Footprint" "Taps Keyboard shit:SW_Cherry_MX_1.00u_PCB"
+		(property "Footprint" "KEYS:SW_Hotswap_Kailh_MX"
 			(at 85.09 59.69 0)
 			(effects
@@
 			)
 		)
-		(property "Footprint" "Taps Keyboard shit:SW_Cherry_MX_1.00u_PCB"
+		(property "Footprint" "KEYS:SW_Hotswap_Kailh_MX"
 			(at 39.37 100.33 0)
 			(effects
@@
 			)
 		)
-		(property "Footprint" "Taps Keyboard shit:SW_Cherry_MX_1.00u_PCB"
+		(property "Footprint" "KEYS:SW_Hotswap_Kailh_MX"
 			(at 54.61 59.69 0)
 			(effects
@@
 			)
 		)
-		(property "Footprint" "Taps Keyboard shit:SW_Cherry_MX_1.00u_PCB"
+		(property "Footprint" "KEYS:SW_Hotswap_Kailh_MX"
 			(at 100.33 39.37 0)
 			(effects
@@
 			)
 		)
-		(property "Footprint" "Taps Keyboard shit:SW_Cherry_MX_1.00u_PCB"
+		(property "Footprint" "KEYS:SW_Hotswap_Kailh_MX"
 			(at 115.57 80.01 0)
 			(effects
@@
 			)
 		)
-		(property "Footprint" "Taps Keyboard shit:SW_Cherry_MX_1.00u_PCB"
+		(property "Footprint" "KEYS:SW_Hotswap_Kailh_MX"
 			(at 54.61 80.01 0)
 			(effects
@@
 			)
 		)
-		(property "Footprint" "Taps Keyboard shit:SW_Cherry_MX_1.00u_PCB"
+		(property "Footprint" "KEYS:SW_Hotswap_Kailh_MX"
 			(at 85.09 39.37 0)
 			(effects
@@
 			)
 		)
-		(property "Footprint" "Taps Keyboard shit:SW_Cherry_MX_1.00u_PCB"
+		(property "Footprint" "KEYS:SW_Hotswap_Kailh_MX"
 			(at 54.61 100.33 0)
 			(effects
@@
 			)
 		)
-		(property "Footprint" "Taps Keyboard shit:SW_Cherry_MX_1.00u_PCB"
+		(property "Footprint" "KEYS:SW_Hotswap_Kailh_MX"
 			(at 69.85 39.37 0)
 			(effects
@@
 			)
 		)
-		(property "Footprint" "Taps Keyboard shit:SW_Cherry_MX_1.00u_PCB"
+		(property "Footprint" "KEYS:SW_Hotswap_Kailh_MX"
 			(at 85.09 80.01 0)
 			(effects
@@
 			)
 		)
-		(property "Footprint" "Taps Keyboard shit:SW_Cherry_MX_1.00u_PCB"
+		(property "Footprint" "KEYS:SW_Hotswap_Kailh_MX"
 			(at 69.85 80.01 0)
 			(effects
@@
 			)
 		)
-		(property "Footprint" "Taps Keyboard shit:SW_Cherry_MX_1.00u_PCB"
+		(property "Footprint" "KEYS:SW_Hotswap_Kailh_MX"
 			(at 39.37 80.01 0)
 			(effects
@@
 			)
 		)
-		(property "Footprint" "Taps Keyboard shit:SW_Cherry_MX_1.00u_PCB"
+		(property "Footprint" "KEYS:SW_Hotswap_Kailh_MX"
 			(at 69.85 100.33 0)
 			(effects
@@
 			)
 		)
-		(property "Footprint" "Taps Keyboard shit:SW_Cherry_MX_1.00u_PCB"
+		(property "Footprint" "KEYS:SW_Hotswap_Kailh_MX"
 			(at 85.09 100.33 0)
 			(effects
@@
 			)
 		)
-		(property "Footprint" "Taps Keyboard shit:SW_Cherry_MX_1.00u_PCB"
+		(property "Footprint" "KEYS:SW_Hotswap_Kailh_MX"
 			(at 39.37 59.69 0)
 			(effects
@@
 			)
 		)
-		(property "Footprint" "Taps Keyboard shit:SW_Cherry_MX_1.00u_PCB"
+		(property "Footprint" "KEYS:SW_Hotswap_Kailh_MX"
 			(at 115.57 59.69 0)
 			(effects
@@
 			)
 		)
-		(property "Footprint" "Taps Keyboard shit:SW_Cherry_MX_1.00u_PCB"
+		(property "Footprint" "KEYS:SW_Hotswap_Kailh_MX"
 			(at 100.33 100.33 0)
 			(effects
@@
 			)
 		)
-		(property "Footprint" "Taps Keyboard shit:SW_Cherry_MX_1.00u_PCB"
+		(property "Footprint" "KEYS:SW_Hotswap_Kailh_MX"
 			(at 54.61 39.37 0)
 			(effects
@@
 			)
 		)
-		(property "Footprint" "Taps Keyboard shit:SW_Cherry_MX_1.00u_PCB"
+		(property "Footprint" "KEYS:SW_Hotswap_Kailh_MX"
 			(at 115.57 100.33 0)
 			(effects

Commit message: Updated Firmware
Parts:
- removed U2: XIAO-nRF52840-DIP, XIAO:XIAO-nRF52840-DIP, symbol XIAO:XIAO-nRF52840-DIP
- added U1: XIAO-RP2350-DIP, Module:MOUDLE14P-XIAO-DIP-SMD, symbol Mitosis:XIAO-RP2350-DIP
Connections:
- net Col10: now also U1.9 (GPIO2/D8/SPI0_SCK)
- net Col11: now also U1.10 (GPIO4/D9/SPI_MISO)
- net Col6: now also U1.5 (GPIO6/D4/SDA1)
- net Col7: now also U1.6 (GPIO7/D5/SCL1)
- net Col8: now also U1.7 (GPIO0/D6/TX0)
- net Col9: now also U1.8 (GPIO1/D7/RX0)
- net Row4: now also U1.1 (GPIO26/D0/ADC0)
- net Row5: now also U1.2 (GPIO27/D1/ADC1)
- net Row6: now also U1.3 (GPIO28/D2/ADC2)
- net Row7: now also U1.4 (GPIO5/D3/SPI_CS)
Changed lines of the file:
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@@
+	)
+	(symbol
+		(lib_id "Mitosis:XIAO-RP2350-DIP")
+		(at 152.4 33.02 0)
+		(unit 1)
+		(exclude_from_sim no)
+		(in_bom yes)
+		(on_board yes)
+		(dnp no)
+		(fields_autoplaced yes)
+		(property "Reference" "U1"
+			(at 167.64 29.21 0)
+			(effects
+				(font
+					(size 1.27 1.27)
+				)
+			)
+		)
+		(property "Value" "XIAO-RP2350-DIP"
+			(at 167.64 31.75 0)
+			(effects
+				(font
+					(size 1.27 1.27)
+				)
+			)
+		)
+		(property "Footprint" "Module:MOUDLE14P-XIAO-DIP-SMD"
+			(at 164.084 63.754 0)
+			(effects
+				(font
+					(size 1.27 1.27)
+				)
+				(hide yes)
+			)
+		)
+		(property "Datasheet" ""
+			(at 152.4 33.02 0)
+			(effects
+				(font
+					(size 1.27 1.27)
+				)
+				(hide yes)
+			)
+		)
+		(property "Description" ""
+			(at 152.4 33.02 0)
+			(effects
+				(font
+					(size 1.27 1.27)
+				)
+				(hide yes)
+			)
+		)
+		(pin "9"
+		)
+		(pin "8"
+		)
+		(pin "10"
+		)
+		(pin "11"
+		)
+		(pin "7"
+		)
+		(pin "13"
+		)
+		(pin "6"
+		)
+		(pin "5"
+		)
+		(pin "4"
+		)
+		(pin "3"
+		)
+		(pin "2"
+		)
+		(pin "1"
+		)
+		(pin "14"
+		)
+		(pin "12"
+		)
+		(instances
+			(project ""
+				(path "/84fc5f43-cc48-4c9a-8e66-78375259861b/774c4cad-5f88-4175-99c1-6b6d60cc7b91"
+					(reference "U1")
+					(unit 1)
+				)
+			)
+		)
 	)
 	(symbol
@@
 					(unit 1)
 				)
-			)
-		)
-	)
-	(symbol
-		(lib_id "XIAO:XIAO-nRF52840-DIP")
-		(at 149.86 33.02 0)
-		(unit 1)
-		(exclude_from_sim no)
-		(in_bom yes)
-		(on_board yes)
-		(dnp no)
-		(fields_autoplaced yes)
-		(property "Reference" "U2"
-			(at 167.64 29.21 0)
-			(effects
-				(font
-					(size 1.27 1.27)
-				)
-			)
-		)
-		(property "Value" "XIAO-nRF52840-DIP"
-			(at 167.64 31.75 0)
-			(effects
-				(font
-					(size 1.27 1.27)
-				)
-			)
-		)
-		(property "Footprint" "XIAO:XIAO-nRF52840-DIP"
-			(at 162.56 63.754 0)
-			(effects
-				(font
-					(size 1.27 1.27)
-				)
-				(hide yes)
-			)
-		)
-		(property "Datasheet" ""
-			(at 146.05 30.48 0)
-			(effects
-				(font
-					(size 1.27 1.27)
-				)
-				(hide yes)
-			)
-		)
-		(property "Description" ""
-			(at 146.05 30.48 0)
-			(effects
-				(font
-					(size 1.27 1.27)
-				)
-				(hide yes)
-			)
-		)
-		(pin "10"
-		)
-		(pin "5"
-		)
-		(pin "6"
-		)
-		(pin "8"
-		)
-		(pin "9"
-		)
-		(pin "12"
-		)
-		(pin "4"
-		)
-		(pin "3"
-		)
-		(pin "2"
-		)
-		(pin "14"
-		)
-		(pin "1"
-		)
-		(pin "13"
-		)
-		(pin "7"
-		)
-		(pin "11"
-		)
-		(instances
-			(project "Tao Te Ching"
-				(path "/84fc5f43-cc48-4c9a-8e66-78375259861b/774c4cad-5f88-4175-99c1-6b6d60cc7b91"
-					(reference "U2")
-					(unit 1)
-				)
