File: PCB/left  sheet.kicad_sch (KiCad schematic)
At the start: 52 parts, among them SW1 SW_Push_45deg, SW10 SW_Push_45deg, SW11 SW_Push_45deg, SW12 SW_Push_45deg, SW13 SW_Push_45deg, SW14 SW_Push_45deg, SW15 SW_Push_45deg, SW16 SW_Push_45deg, SW17 SW_Push_45deg, SW18 SW_Push_45deg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

Commit message: Added hotswap sockets
Parts:
- SW1, SW10, SW11, SW12, SW13, SW14, SW15, SW16, SW17, SW18, SW19, SW2, SW20, SW21, SW22, SW23, SW24, SW3, SW4, SW5, SW6, SW7, SW8, SW9: footprint Taps Keyboard shit:SW_Cherry_MX_1.00u_PCB -> KEYS:SW_Hotswap_Kailh_MX
Changed lines of the file:
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@@
 			)
 		)
-		(property "Footprint" "Taps Keyboard shit:SW_Cherry_MX_1.00u_PCB"
+		(property "Footprint" "KEYS:SW_Hotswap_Kailh_MX"
 			(at 60.96 92.71 0)
 			(effects
@@
 			)
 		)
-		(property "Footprint" "Taps Keyboard shit:SW_Cherry_MX_1.00u_PCB"
+		(property "Footprint" "KEYS:SW_Hotswap_Kailh_MX"
 			(at 60.96 52.07 0)
 			(effects
@@
 			)
 		)
-		(property "Footprint" "Taps Keyboard shit:SW_Cherry_MX_1.00u_PCB"
+		(property "Footprint" "KEYS:SW_Hotswap_Kailh_MX"
 			(at 106.68 113.03 0)
 			(effects
@@
 			)
 		)
-		(property "Footprint" "Taps Keyboard shit:SW_Cherry_MX_1.00u_PCB"
+		(property "Footprint" "KEYS:SW_Hotswap_Kailh_MX"
 			(at 121.92 52.07 0)
 			(effects
@@
 			)
 		)
-		(property "Footprint" "Taps Keyboard shit:SW_Cherry_MX_1.00u_PCB"
+		(property "Footprint" "KEYS:SW_Hotswap_Kailh_MX"
 			(at 76.2 92.71 0)
 			(effects
@@
 			)
 		)
-		(property "Footprint" "Taps Keyboard shit:SW_Cherry_MX_1.00u_PCB"
+		(property "Footprint" "KEYS:SW_Hotswap_Kailh_MX"
 			(at 91.44 92.71 0)
 			(effects
@@
 			)
 		)
-		(property "Footprint" "Taps Keyboard shit:SW_Cherry_MX_1.00u_PCB"
+		(property "Footprint" "KEYS:SW_Hotswap_Kailh_MX"
 			(at 121.92 113.03 0)
 			(effects
@@
 			)
 		)
-		(property "Footprint" "Taps Keyboard shit:SW_Cherry_MX_1.00u_PCB"
+		(property "Footprint" "KEYS:SW_Hotswap_Kailh_MX"
 			(at 121.92 72.39 0)
 			(effects
@@
 			)
 		)
-		(property "Footprint" "Taps Keyboard shit:SW_Cherry_MX_1.00u_PCB"
+		(property "Footprint" "KEYS:SW_Hotswap_Kailh_MX"
 			(at 106.68 92.71 0)
 			(effects
@@
 			)
 		)
-		(property "Footprint" "Taps Keyboard shit:SW_Cherry_MX_1.00u_PCB"
+		(property "Footprint" "KEYS:SW_Hotswap_Kailh_MX"
 			(at 76.2 72.39 0)
 			(effects
@@
 			)
 		)
-		(property "Footprint" "Taps Keyboard shit:SW_Cherry_MX_1.00u_PCB"
+		(property "Footprint" "KEYS:SW_Hotswap_Kailh_MX"
 			(at 91.44 72.39 0)
 			(effects
@@
 			)
 		)
-		(property "Footprint" "Taps Keyboard shit:SW_Cherry_MX_1.00u_PCB"
+		(property "Footprint" "KEYS:SW_Hotswap_Kailh_MX"
 			(at 76.2 113.03 0)
 			(effects
@@
 			)
 		)
-		(property "Footprint" "Taps Keyboard shit:SW_Cherry_MX_1.00u_PCB"
+		(property "Footprint" "KEYS:SW_Hotswap_Kailh_MX"
 			(at 106.68 72.39 0)
 			(effects
@@
 			)
 		)
-		(property "Footprint" "Taps Keyboard shit:SW_Cherry_MX_1.00u_PCB"
+		(property "Footprint" "KEYS:SW_Hotswap_Kailh_MX"
 			(at 45.72 113.03 0)
 			(effects
@@
 			)
 		)
-		(property "Footprint" "Taps Keyboard shit:SW_Cherry_MX_1.00u_PCB"
+		(property "Footprint" "KEYS:SW_Hotswap_Kailh_MX"
 			(at 121.92 92.71 0)
 			(effects
@@
 			)
 		)
-		(property "Footprint" "Taps Keyboard shit:SW_Cherry_MX_1.00u_PCB"
+		(property "Footprint" "KEYS:SW_Hotswap_Kailh_MX"
 			(at 91.44 52.07 0)
 			(effects
@@
 			)
 		)
-		(property "Footprint" "Taps Keyboard shit:SW_Cherry_MX_1.00u_PCB"
+		(property "Footprint" "KEYS:SW_Hotswap_Kailh_MX"
 			(at 45.72 92.71 0)
 			(effects
@@
 			)
 		)
-		(property "Footprint" "Taps Keyboard shit:SW_Cherry_MX_1.00u_PCB"
+		(property "Footprint" "KEYS:SW_Hotswap_Kailh_MX"
 			(at 60.96 72.39 0)
 			(effects
@@
 			)
 		)
-		(property "Footprint" "Taps Keyboard shit:SW_Cherry_MX_1.00u_PCB"
+		(property "Footprint" "KEYS:SW_Hotswap_Kailh_MX"
 			(at 106.68 52.07 0)
 			(effects
@@
 			)
 		)
-		(property "Footprint" "Taps Keyboard shit:SW_Cherry_MX_1.00u_PCB"
+		(property "Footprint" "KEYS:SW_Hotswap_Kailh_MX"
 			(at 76.2 52.07 0)
 			(effects
@@
 			)
 		)
-		(property "Footprint" "Taps Keyboard shit:SW_Cherry_MX_1.00u_PCB"
+		(property "Footprint" "KEYS:SW_Hotswap_Kailh_MX"
 			(at 60.96 113.03 0)
 			(effects
@@
 			)
 		)
-		(property "Footprint" "Taps Keyboard shit:SW_Cherry_MX_1.00u_PCB"
+		(property "Footprint" "KEYS:SW_Hotswap_Kailh_MX"
 			(at 45.72 72.39 0)
 			(effects
@@
 			)
 		)
-		(property "Footprint" "Taps Keyboard shit:SW_Cherry_MX_1.00u_PCB"
+		(property "Footprint" "KEYS:SW_Hotswap_Kailh_MX"
 			(at 91.44 113.03 0)
 			(effects
@@
 			)
 		)
-		(property "Footprint" "Taps Keyboard shit:SW_Cherry_MX_1.00u_PCB"
+		(property "Footprint" "KEYS:SW_Hotswap_Kailh_MX"
 			(at 45.72 52.07 0)
 			(effects

Commit message: Updated Firmware
Parts:
- removed U1: XIAO-nRF52840-DIP, XIAO:XIAO-nRF52840-DIP, symbol XIAO:XIAO-nRF52840-DIP
- added U3: XIAO-RP2350-DIP, Module:MOUDLE14P-XIAO-DIP-SMD, symbol Mitosis:XIAO-RP2350-DIP
Connections:
- net Col0: now also U3.5 (GPIO6/D4/SDA1)
- net Col1: now also U3.6 (GPIO7/D5/SCL1)
- net Col2: now also U3.7 (GPIO0/D6/TX0)
- net Col3: now also U3.10 (GPIO4/D9/SPI_MISO)
- net Col4: now also U3.9 (GPIO2/D8/SPI0_SCK)
- net Col5: now also U3.8 (GPIO1/D7/RX0)
- net Row0: now also U3.1 (GPIO26/D0/ADC0)
- net Row1: now also U3.2 (GPIO27/D1/ADC1)
- net Row2: now also U3.3 (GPIO28/D2/ADC2)
- net Row3: now also U3.4 (GPIO5/D3/SPI_CS)
Changed lines of the file:
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@@
-	)
-	(symbol
-		(lib_id "XIAO:XIAO-nRF52840-DIP")
-		(at 157.48 46.99 0)
-		(unit 1)
-		(exclude_from_sim no)
-		(in_bom yes)
-		(on_board yes)
-		(dnp no)
-		(fields_autoplaced yes)
-		(property "Reference" "U1"
-			(at 175.26 43.18 0)
-			(effects
-				(font
-					(size 1.27 1.27)
-				)
-			)
-		)
-		(property "Value" "XIAO-nRF52840-DIP"
-			(at 175.26 45.72 0)
-			(effects
-				(font
-					(size 1.27 1.27)
-				)
-			)
-		)
-		(property "Footprint" "XIAO:XIAO-nRF52840-DIP"
-			(at 170.18 77.724 0)
-			(effects
-				(font
-					(size 1.27 1.27)
-				)
-				(hide yes)
-			)
-		)
-		(property "Datasheet" ""
-			(at 153.67 44.45 0)
-			(effects
-				(font
-					(size 1.27 1.27)
-				)
-				(hide yes)
-			)
-		)
-		(property "Description" ""
-			(at 153.67 44.45 0)
-			(effects
-				(font
-					(size 1.27 1.27)
-				)
-				(hide yes)
-			)
-		)
-		(pin "10"
-		)
-		(pin "5"
-		)
-		(pin "6"
-		)
-		(pin "8"
-		)
-		(pin "9"
-		)
-		(pin "12"
-		)
-		(pin "4"
-		)
-		(pin "3"
-		)
-		(pin "2"
-		)
-		(pin "14"
-		)
-		(pin "1"
-		)
-		(pin "13"
-		)
-		(pin "7"
-		)
-		(pin "11"
-		)
-		(instances
-			(project ""
-				(path "/84fc5f43-cc48-4c9a-8e66-78375259861b/0d265e0a-c39a-494d-aa60-6f642baae709"
-					(reference "U1")
-					(unit 1)
-				)
-			)
-		)
 	)
 	(symbol
@@
 					(unit 1)
 				)
+			)
+		)
+	)
+	(symbol
+		(lib_id "Mitosis:XIAO-RP2350-DIP")
+		(at 160.02 46.99 0)
+		(unit 1)
+		(exclude_from_sim no)
+		(in_bom yes)
+		(on_board yes)
+		(dnp no)
+		(fields_autoplaced yes)
+		(property "Reference" "U3"
+			(at 175.26 43.18 0)
+			(effects
+				(font
+					(size 1.27 1.27)
+				)
+			)
+		)
+		(property "Value" "XIAO-RP2350-DIP"
+			(at 175.26 45.72 0)
+			(effects
+				(font
+					(size 1.27 1.27)
+				)
+			)
+		)
+		(property "Footprint" "Module:MOUDLE14P-XIAO-DIP-SMD"
+			(at 171.704 77.724 0)
+			(effects
+				(font
+					(size 1.27 1.27)
+				)
+				(hide yes)
+			)
+		)
+		(property "Datasheet" ""
+			(at 160.02 46.99 0)
+			(effects
+				(font
+					(size 1.27 1.27)
+				)
+				(hide yes)
+			)
+		)
+		(property "Description" ""
+			(at 160.02 46.99 0)
+			(effects
+				(font
+					(size 1.27 1.27)
+				)
+				(hide yes)
+			)
+		)
+		(pin "10"
+		)
+		(pin "13"
+		)
+		(pin "12"
+		)
+		(pin "11"
+		)
+		(pin "9"
+		)
+		(pin "14"
+		)
+		(pin "2"
+		)
+		(pin "3"
+		)
+		(pin "4"
+		)
+		(pin "5"
+		)
+		(pin "6"
+		)
+		(pin "7"
+		)
+		(pin "1"
+		)
+		(pin "8"
+		)
+		(instances
+			(project ""
+				(path "/84fc5f43-cc48-4c9a-8e66-78375259861b/0d265e0a-c39a-494d-aa60-6f642baae709"
+					(reference "U3")
+					(unit 1)
+				)
